Commit message: teleop movement added

File: src/ros_project_scene/urdf/robot_model.xacro (robot description, xacro)
@@ -36,5 +36,5 @@
             <material name="white"/>
         </visual>
-        <xacro:inertial_box mass="1" x="0.2" y="0.6" z="0.6">
+        <xacro:inertial_box mass="2" x="0.2" y="0.6" z="0.6">
             <origin xyz="0 0 0.2" rpy="0 ${pi/2} 0"/>
         </xacro:inertial_box>
@@ -92,9 +92,8 @@
         </inertial>
     </link>
-    <joint name="camera_joint" type="continuous">
+    <joint name="camera_joint" type="fixed">
         <origin xyz="0.275 0 0.37" rpy="0 0 0"/>
         <parent link="base_link"/>
         <child link="camera_link"/>
-        <axis xyz="0 0 1"/>
     </joint>
     <gazebo reference="camera_link">
@@ -143,9 +142,8 @@
         </collision>
     </link>
-    <joint name="lidar_joint" type="continuous">
+    <joint name="lidar_joint" type="fixed">
         <origin xyz="0.275 0 0.325" rpy="0 0 0"/>
         <child link="lidar_link"/>
         <parent link="base_link"/>
-        <axis xyz="0 0 1"/>
     </joint>
     <gazebo reference="lidar_link">

Commit message: final results

File: src/ros_project_scene/urdf/robot_model.xacro (robot description, xacro)
@@ -93,6 +93,6 @@
     </link>
     <joint name="camera_joint" type="fixed">
-        <origin xyz="0.275 0 0.37" rpy="0 0 0"/>
-        <parent link="base_link"/>
+        <origin xyz="0.01 0 0.06" rpy="0 0.5 0"/>
+        <parent link="lidar_link"/>
         <child link="camera_link"/>
     </joint>
@@ -102,5 +102,5 @@
             <pose> 0 0 0 0 0 0 </pose>
             <visualize>true</visualize>
-            <update_rate>10</update_rate>
+            <update_rate>15</update_rate>
             <camera>
                 <camera_info_topic>camera/camera_info</camera_info_topic>
